File: kicad/spectrum/front_panel/front_panel.kicad_pcb (KiCad board)
At the start: 2 copper layers, 248.5 x 36 mm, 78 parts, among them J1 SSD1322, J10 SWD, J2 POWER, J3 I2C, J4 UART, J5 EXT_INPUT, J6 AUDIO, J7 SYNC, J8 SPI, J9 CONTROL, SW1 ST1, SW10 BAND, SW11 RDS, SW12 FM_ENC, SW13 MENU, SW14 RST, SW2 ST4, SW3 ST7, SW4 ST2, SW5 ST5, SW6 ST8, SW7 ST3, SW8 ST6, SW9 ST9, U1 STM32F303CCTx, U2 MCP602, U3 AMS1117-3.3, U4 AMS1117-3.3, U5 TSOP4538, Y1 8MHz, Y2 32768

Commit message: Change to STM32F103CB in Kicad project
Parts:
- U1: value STM32F303CCTx -> STM32F103CBTx
Changed lines of the file:
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@@
-(kicad_pcb (version 20171130) (host pcbnew 5.1.4)
+(kicad_pcb (version 20171130) (host pcbnew 5.1.5)
   (general
     (thickness 1.6)
@@
       (effects (font (size 1 1) (thickness 0.15)) (justify mirror))
     )
-    (fp_text value STM32F303CCTx (at 4.25 7.25 180) (layer B.SilkS)
+    (fp_text value STM32F103CBTx (at 4.25 7.25 180) (layer B.SilkS)
       (effects (font (size 1 1) (thickness 0.15)) (justify mirror))
     )

Commit message: Update schematcis and PCB
Parts:
- added C21: 2.2, Capacitor_SMD:C_1206_3216Metric_Pad1.42x1.75mm_HandSolder, B.Cu at (132.9, 109.9)
- added C22: 2.2, Capacitor_SMD:C_1206_3216Metric_Pad1.42x1.75mm_HandSolder, B.Cu at (126.8, 109.9)
- moved R16 3.12 mm to (136.8, 108.8), turned to 90 degrees
- moved R17 2.77 mm to (122.6, 108.8), turned to 90 degrees
- moved R13 0.73 mm to (123.2, 103.3)
- moved R12 0.71 mm to (135.9, 103.3)
- moved C8 0.14 mm to (140.1, 121.9)
- moved C9 0.08 mm to (122.8, 121.9)
Connections:
- R16 pad 1: Net-(R16-Pad1) -> Net-(C21-Pad1)
- R17 pad 1: Net-(R17-Pad1) -> Net-(C22-Pad1)
- RV1 pad 2: Net-(R16-Pad1) -> Net-(C21-Pad2)
- RV2 pad 2: Net-(R17-Pad1) -> Net-(C22-Pad2)
Routing:
- net Net-(C22-Pad2): track 0.00 -> 5.84 mm
- net Net-(C21-Pad2): track 0.00 -> 5.30 mm
- net Net-(R16-Pad1): track 4.91 -> 0.00 mm
- net Net-(R17-Pad1): track 4.80 -> 0.00 mm
- net Net-(R13-Pad1): track 10.5 -> 6.62 mm
- net Net-(C22-Pad1): track 0.00 -> 2.92 mm
- net Net-(C21-Pad1): track 0.00 -> 2.54 mm
- net +5V: track 267.6 -> 269.4 mm
- net Net-(R12-Pad1): track 9.21 -> 7.37 mm
- net /SP_R: track 34.9 -> 33.7 mm
- net +3V3: track 327.9 -> 327.2 mm
- net /DISP_RST: track 81.9 -> 82.4 mm
- net /DISP_DIN: track 84.0 -> 84.5 mm
- net /DISP_DC: track 92.6 -> 93.1 mm
- net /DISP_CS: track 101.6 -> 101.1 mm
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