File: kicad/common/front_panel/front_panel.kicad_pcb (KiCad board)
At the start: 2 copper layers, 248.5 x 36 mm, 80 parts, among them J1 SSD1322, J10 SWD, J2 POWER, J3 I2C, J4 UART, J5 EXT_INPUT, J6 AUDIO, J7 SYNC, J8 SPI, J9 CONTROL, SW1 ST1, SW10 BAND, SW11 RDS, SW12 FM_ENC, SW13 MENU, SW14 RST, SW2 ST4, SW3 ST7, SW4 ST2, SW5 ST5, SW6 ST8, SW7 ST3, SW8 ST6, SW9 ST9, U1 STM32F103CBTx, U2 MCP602, U3 AMS1117-3.3, U4 AMS1117-3.3, U5 TSOP4538, Y1 8MHz, Y2 32768

Commit message: Update schematics
Parts:
- C1, C11, C12, C13, C14, C17, C18, C19, C2, C20, C21, C22, C3, C4, C5, C6, C7, C8, C9: footprint Capacitor_SMD:C_1206_3216Metric_Pad1.42x1.75mm_HandSolder -> Capacitor_SMD:C_1206_3216Metric_Pad1.33x1.80mm_HandSolder
- R1, R10, R11, R12, R13, R14, R15, R16, R17, R18, R19, R2, R20, R21, R3, R4, R5, R6, R7, R8, R9: footprint Resistor_SMD:R_1206_3216Metric_Pad1.42x1.75mm_HandSolder -> Resistor_SMD:R_1206_3216Metric_Pad1.30x1.75mm_HandSolder

Commit message: Move common front panel to Kicad 6
Other:
- net class Default removed
