File: kicad/player/front_panel/front_panel.kicad_pcb (KiCad board)
At the start: 2 copper layers, 253 x 38.5 mm, 59 parts, among them J1 SSD1322, J10 SWD, J11 USB, J2 POWER, J3 I2C, J4 UART, J5 EXT_INPUT, J6 ENCODER, J7 SYNC, J8 SPI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

Commit message: Update schematics
Parts:
- C11, C12, C13, C14, C17, C18, C19, C20, C3, C4, C5, C6, C7: footprint Capacitor_SMD:C_1206_3216Metric_Pad1.42x1.75mm_HandSolder -> Capacitor_SMD:C_1206_3216Metric_Pad1.33x1.80mm_HandSolder
- R1, R10, R11, R18, R19, R2, R20, R21, R3, R4, R5, R6, R7: footprint Resistor_SMD:R_1206_3216Metric_Pad1.42x1.75mm_HandSolder -> Resistor_SMD:R_1206_3216Metric_Pad1.30x1.75mm_HandSolder
- R8: value 1.5k -> 10k; footprint Resistor_SMD:R_1206_3216Metric_Pad1.42x1.75mm_HandSolder -> Resistor_SMD:R_1206_3216Metric_Pad1.30x1.75mm_HandSolder
- moved R6 0.14 mm to (203.8, 109.5)
- moved R7 0.14 mm to (207.6, 109.5)
- moved R8 0.14 mm to (211.5, 109.5)
- moved R20 0.06 mm to (182.9, 105.7)
- moved R21 0.06 mm to (179.1, 105.7)

Commit message: Update player front_panel to Kicad 7
Other:
- net class Default removed
